File: KiCAD/Thermometry.kicad_pcb (KiCad board)
At the start: 2 copper layers, 50 parts, among them J1 Barrel_Jack_Switch, J2 DB15_Female_MountingHoles, J3 RJ45_LED_Shielded, J4 Conn_01x02_Female, J5 Conn_01x02_Female, U1 MAX31865, U2 MAX31865, U3 MAX31865, U4 MAX31865, U5 MAX31865, U6 Teensy4.1, U7 MAX31856, U8 MAX31856, U9 MAX31723

Commit message: routing progress
Parts:
- C1, C11, C12, C13, C14, C15, C16, C17, C18, C19, C2, C20, C21, C22, C23, C24, C25, C26, C27, C28, C29, C3, C4, C5, C6, C7, C8, C9: footprint Capacitor_SMD:C_0805_2012Metric_Pad1.15x1.40mm_HandSolder -> Capacitor_SMD:C_0805_2012Metric_Pad1.18x1.45mm_HandSolder
- J2: footprint Connector_Dsub:DSUB-15-HD_Female_Horizontal_P2.29x1.98mm_EdgePinOffset3.03mm_Housed_MountingHolesOffset4.94mm -> Connector_Dsub:DSUB-15_Male_Horizontal_P2.77x2.84mm_EdgePinOffset4.94mm_Housed_MountingHolesOffset7.48mm
- J4, J5: footprint Connector_Wire:SolderWire-0.15sqmm_1x02_P4mm_D0.5mm_OD1.5mm_Relief2x -> Connector_Wire:SolderWire-0.15sqmm_1x02_P4mm_D0.5mm_OD1.5mm
- R1, R2, R3, R4, R5: footprint Resistor_SMD:R_1206_3216Metric_Pad1.42x1.75mm_HandSolder -> Resistor_SMD:R_1206_3216Metric_Pad1.30x1.75mm_HandSolder
- R6, R7: footprint Resistor_SMD:R_0805_2012Metric_Pad1.15x1.40mm_HandSolder -> Resistor_SMD:R_0805_2012Metric_Pad1.20x1.40mm_HandSolder
- moved C14 96.5 mm to (134.9, 48.0), turned to 90 degrees
- moved C20 81.1 mm to (96.2, 24.1)
- moved J2 76.2 mm to (144.0, 73.4), turned to 90 degrees
- moved C12 67.5 mm to (125.2, 78.8), turned to 90 degrees
- moved U5 67.2 mm to (129.5, 56.4), turned to 90 degrees
- moved J4 67.0 mm to (138.2, 26.7), turned to 90 degrees
- moved U8 66.2 mm to (111.8, 32.9)
- moved C18 65.4 mm to (90.1, 24.6)
- moved R5 64.1 mm to (163.5, 88.7)
- moved U7 58.2 mm to (97.8, 32.5)
- moved J5 58.2 mm to (138.2, 35.1), turned to 90 degrees
- moved C25 58.0 mm to (87.7, 31.3)
- moved C10 55.8 mm to (76.7, 37.1), turned to 270 degrees
- moved J1 53.6 mm to (70.1, 32.0)
- moved C26 51.4 mm to (101.4, 23.8)
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Routing:
- net +3V3: track 0.00 -> 193.1 mm
- net GND: track 0.00 -> 67.4 mm, vias 0 -> 10
- net Net-(C10-Pad1): track 0.00 -> 32.6 mm
- net SCLK: track 0.00 -> 29.1 mm, vias 0 -> 2
- net SDI: track 0.00 -> 15.4 mm, vias 0 -> 2
- net SDO: track 0.00 -> 10.6 mm, vias 0 -> 1
- net RTD3_N: track 0.00 -> 7.45 mm, vias 0 -> 1
- net RTD2_N: track 0.00 -> 6.95 mm
- net Net-(R3-Pad2): track 0.00 -> 6.84 mm
- net RTD1_N: track 0.00 -> 6.81 mm
- net Net-(R2-Pad2): track 0.00 -> 6.71 mm
- net RTD2_P: track 0.00 -> 6.37 mm
- net Net-(R1-Pad2): track 0.00 -> 6.18 mm
- net RTD1_P: track 0.00 -> 6.16 mm
- net Net-(R4-Pad2): track 0.00 -> 6.10 mm
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- added copper zone on B.Cu, net GND
Other:
- copper layers 2 -> 4
