File: KiCAD/Thermometry.sch (KiCad schematic (older format))
At the start: 50 parts, among them J1 Barrel_Jack_Switch, J2 DB15_Female_MountingHoles, J3 RJ45_LED_Shielded, J4 Conn_01x02_Female, J5 Conn_01x02_Female, U1 MAX31865, U2 MAX31865, U3 MAX31865, U4 MAX31865, U5 MAX31865, U6 Teensy4.1, U7 MAX31856, U8 MAX31856, U9 MAX31723

Commit message: updated sch and netlists for PCB placements
Parts:
- C10: footprint (none) -> Capacitor_THT:CP_Radial_D5.0mm_P2.00mm
- J1: footprint Connector_BarrelJack:BarrelJack_CUI_PJ-063AH_Horizontal -> Connector_BarrelJack:BarrelJack_Horizontal
- J3: symbol Connector:RJ45_LED_Shielded -> ThermoLib:8P8C_LED_Shielded
- U1, U2, U3, U4, U5: footprint ThermometryFull:SOIC-20 -> Thermometry:MAX31865
- U6: footprint (none) -> Thermometry:Teensy41; symbol _MyLib_Teensy:Teensy4.1 -> ThermoLib:Teensy4.1
- U7, U8: footprint (none) -> Thermometry:MAX31856
- U9: footprint (none) -> Thermometry:MAX3172X
Connections:
- net GND: now also J3.13
- no-connect marks 54 -> 40
Changed lines of the file:
@@
 F 0 "U1" H 6425 2665 50  0000 C CNN
 F 1 "MAX31865" H 6425 2574 50  0000 C CNN
-F 2 "ThermometryFull:SOIC-20" H 6350 1900 50  0001 C CNN
+F 2 "Thermometry:MAX31865" H 6350 1900 50  0001 C CNN
 F 3 "https://datasheets.maximintegrated.com/en/ds/MAX31865.pdf" H 6350 1900 50  0001 C CNN
 F 4 "MAX31865AAP+TCT-ND" H 6450 1900 50  0001 C CNN "DigikeyPN"
@@
 F 0 "U2" H 8925 2665 50  0000 C CNN
 F 1 "MAX31865" H 8925 2574 50  0000 C CNN
-F 2 "ThermometryFull:SOIC-20" H 8850 1900 50  0001 C CNN
+F 2 "Thermometry:MAX31865" H 8850 1900 50  0001 C CNN
 F 3 "https://datasheets.maximintegrated.com/en/ds/MAX31865.pdf" H 8850 1900 50  0001 C CNN
 F 4 "MAX31865AAP+TCT-ND" H 8950 1900 50  0001 C CNN "DigikeyPN"
@@
 F 0 "U3" H 11425 2665 50  0000 C CNN
 F 1 "MAX31865" H 11425 2574 50  0000 C CNN
-F 2 "ThermometryFull:SOIC-20" H 11350 1900 50  0001 C CNN
+F 2 "Thermometry:MAX31865" H 11350 1900 50  0001 C CNN
 F 3 "https://datasheets.maximintegrated.com/en/ds/MAX31865.pdf" H 11350 1900 50  0001 C CNN
 F 4 "MAX31865AAP+TCT-ND" H 11450 1900 50  0001 C CNN "DigikeyPN"
@@
 F 0 "U4" H 6425 4665 50  0000 C CNN
 F 1 "MAX31865" H 6425 4574 50  0000 C CNN
-F 2 "ThermometryFull:SOIC-20" H 6350 3900 50  0001 C CNN
+F 2 "Thermometry:MAX31865" H 6350 3900 50  0001 C CNN
 F 3 "https://datasheets.maximintegrated.com/en/ds/MAX31865.pdf" H 6350 3900 50  0001 C CNN
 F 4 "MAX31865AAP+TCT-ND" H 6450 3900 50  0001 C CNN "DigikeyPN"
@@
 F 0 "U5" H 8925 4665 50  0000 C CNN
 F 1 "MAX31865" H 8925 4574 50  0000 C CNN
-F 2 "ThermometryFull:SOIC-20" H 8850 3900 50  0001 C CNN
+F 2 "Thermometry:MAX31865" H 8850 3900 50  0001 C CNN
 F 3 "https://datasheets.maximintegrated.com/en/ds/MAX31865.pdf" H 8850 3900 50  0001 C CNN
 F 4 "MAX31865AAP+TCT-ND" H 8950 3900 50  0001 C CNN "DigikeyPN"
@@
 F 0 "J1" H 2907 1767 50  0000 C CNN
 F 1 "Barrel_Jack_Switch" H 2907 1676 50  0000 C CNN
-F 2 "Connector_BarrelJack:BarrelJack_CUI_PJ-063AH_Horizontal" H 2900 1410 50  0001 C CNN
+F 2 "Connector_BarrelJack:BarrelJack_Horizontal" H 2900 1410 50  0001 C CNN
 F 3 "https://www.cuidevices.com/product/resource/pj-002a.pdf" H 2900 1410 50  0001 C CNN
 F 4 "CP-002A-ND" H 2850 1450 50  0001 C CNN "DigikeyPN"
@@
 $EndComp
 $Comp
-L Connector:RJ45_LED_Shielded J3
+L ThermoLib:8P8C_LED_Shielded J3
 U 1 1 6155BBE8
 P 2750 7050
@@
 	3700 5350 3700 7350
 Wire Wire Line
-	3650 5450 3250 5450
-Wire Wire Line
 	3150 7350 3700 7350
 Wire Wire Line
-	3250 5350 3700 5350
-Wire Wire Line
 	3150 6650 3600 6650
 Wire Wire Line
 	3600 6650 3600 6350
-Wire Wire Line
-	3600 5250 3250 5250
 Wire Wire Line
 	2350 6650 2300 6650
@@
 Wire Wire Line
 	3500 6850 3500 5650
-Wire Wire Line
-	3500 5650 3250 5650
-Wire Wire Line
-	3250 5550 3350 5550
 Wire Wire Line
 	3350 5550 3350 6250
@@
 F 0 "C10" V 3650 2400 50  0000 C CNN
 F 1 "47uF" V 3550 2300 50  0000 C CNN
-F 2 "" H 3500 2600 50  0001 C CNN
+F 2 "Capacitor_THT:CP_Radial_D5.0mm_P2.00mm" H 3500 2600 50  0001 C CNN
 F 3 "~" H 3500 2600 50  0001 C CNN
 	1    3500 2600
@@
 	3400 1350 3400 2600
 Connection ~ 3400 2600
-Wire Wire Line
-	3250 2700 3600 2700
 Wire Wire Line
 	3600 2600 3600 1550
@@
 	3600 2950 3600 2900
 Wire Wire Line
-	3250 2800 3450 2800
-Wire Wire Line
 	3450 2800 3450 2950
 Wire Wire Line
@@
 F 0 "U7" H 6400 6615 50  0000 C CNN
 F 1 "MAX31856" H 6400 6524 50  0000 C CNN
-F 2 "" H 6200 6250 50  0001 C CNN
+F 2 "Thermometry:MAX31856" H 6200 6250 50  0001 C CNN
 F 3 "https://datasheets.maximintegrated.com/en/ds/MAX31865.pdf" H 6200 6250 50  0001 C CNN
 F 4 "MAX31856MUD+TCT-ND" H 6400 6100 50  0001 C CNN "DigikeyPN"
@@
 F 0 "U8" H 9400 6615 50  0000 C CNN
 F 1 "MAX31856" H 9400 6524 50  0000 C CNN
-F 2 "" H 9200 6250 50  0001 C CNN
+F 2 "Thermometry:MAX31856" H 9200 6250 50  0001 C CNN
 F 3 "https://datasheets.maximintegrated.com/en/ds/MAX31865.pdf" H 9200 6250 50  0001 C CNN
 F 4 "MAX31856MUD+TCT-ND" H 9400 6100 50  0001 C CNN "DigikeyPN"
@@
 F 0 "U9" H 6100 8415 50  0000 C CNN
 F 1 "MAX31723" H 6100 8324 50  0000 C CNN
-F 2 "" H 6050 7950 50  0001 C CNN
+F 2 "Thermometry:MAX3172X" H 6050 7950 50  0001 C CNN
 F 3 "" H 6050 7950 50  0001 C CNN
 	1    6100 8000
@@
 NoConn ~ 2350 7250
 NoConn ~ 2350 7350
-NoConn ~ 2450 6050
-NoConn ~ 2300 6050
-NoConn ~ 2150 6050
-NoConn ~ 2000 6050
-NoConn ~ 1850 6050
-NoConn ~ 2750 7550
-NoConn ~ 1050 5750
-NoConn ~ 1050 5650
-NoConn ~ 1050 5550
-NoConn ~ 1050 5450
-NoConn ~ 1050 5350
-NoConn ~ 1050 5200
-NoConn ~ 1050 5100
 $Comp
 L Device:R_Small_US R6
@@
 	0    -1   -1   0
 $EndComp
-Wire Wire Line
-	3350 3900 3250 3900
 Text GLabel 3600 3900 2    50   Input ~ 0
 SCLK
@@
 	1    0    0    -1
 $EndComp
-Wire Wire Line
-	3250 4000 3500 4000
 $Comp
 L power:GND #PWR0102
@@
 F 3 "" H 6950 8000 50  0001 C CNN
 	1    6950 8000
-	1    0    0    -1
-$EndComp
-Wire Wire Line
-	3550 3100 3250 3100
-Wire Wire Line
-	3550 3200 3250 3200
-Wire Wire Line
-	3550 3300 3250 3300
-Wire Wire Line
-	3550 3400 3250 3400
-Wire Wire Line
-	3550 3500 3250 3500
-Wire Wire Line
-	3450 4700 3250 4700
-Wire Wire Line
-	3450 4600 3250 4600
-Wire Wire Line
-	3450 4500 3250 4500
-Wire Wire Line
-	3450 4400 3250 4400
-Wire Wire Line
-	3450 4300 3250 4300
-$Comp
-L _MyLib_Teensy:Teensy4.1 U6
-U 1 1 614A8781
-P 2150 4750
-F 0 "U6" H 2150 7315 50  0000 C CNN
-F 1 "Teensy4.1" H 2150 7224 50  0000 C CNN
-F 2 "" H 1750 5150 50  0001 C CNN
-F 3 "" H 1750 5150 50  0001 C CNN
-	1    2150 4750
 	1    0    0    -1
 $EndComp
@@
 	3950 5250 3600 5250
 Connection ~ 3600 5250
-NoConn ~ 3250 2450
 NoConn ~ 5700 7850
+$Comp
+L power:GND #PWR0105
+U 1 1 614670CB
+P 2750 7550
+F 0 "#PWR0105" H 2750 7300 50  0001 C CNN
+F 1 "GND" H 2900 7550 50  0000 C CNN
+F 2 "" H 2750 7550 50  0001 C CNN
+F 3 "" H 2750 7550 50  0001 C CNN
+	1    2750 7550
+	1    0    0    -1
+$EndComp
+Wire Wire Line
+	3500 5650 3250 5650
+Wire Wire Line
+	3250 5550 3350 5550
+Wire Wire Line
+	3650 5450 3250 5450
+Wire Wire Line
+	3250 5350 3700 5350
+Wire Wire Line
+	3600 5250 3250 5250
+Wire Wire Line
+	3450 4700 3250 4700
+Wire Wire Line
+	3450 4600 3250 4600
+Wire Wire Line
+	3450 4500 3250 4500
+Wire Wire Line
+	3450 4400 3250 4400
+Wire Wire Line
+	3450 4300 3250 4300
+Wire Wire Line
+	3250 4000 3500 4000
+Wire Wire Line
+	3350 3900 3250 3900
+Wire Wire Line
+	3550 3500 3250 3500
+Wire Wire Line
+	3550 3400 3250 3400
+Wire Wire Line
+	3550 3300 3250 3300
+Wire Wire Line
+	3550 3200 3250 3200
+Wire Wire Line
+	3550 3100 3250 3100
+Wire Wire Line
+	3250 2800 3450 2800
+Wire Wire Line
+	3250 2700 3600 2700
+$Comp
+L ThermoLib:Teensy4.1 U6
+U 1 1 614A8781
+P 2150 4750
+F 0 "U6" H 2150 7315 50  0000 C CNN
+F 1 "Teensy4.1" H 2150 7224 50  0000 C CNN
+F 2 "Thermometry:Teensy41" H 1750 5150 50  0001 C CNN
+F 3 "" H 1750 5150 50  0001 C CNN
+	1    2150 4750
+	1    0    0    -1
+$EndComp
 $EndSCHEMATC

Commit message: routing progress
Parts:
- C1, C11, C12, C13, C14, C15, C16, C17, C18, C19, C2, C20, C21, C22, C23, C24, C25, C26, C27, C28, C29, C3, C4, C5, C6, C7, C8, C9: footprint Capacitor_SMD:C_0805_2012Metric_Pad1.15x1.40mm_HandSolder -> Capacitor_SMD:C_0805_2012Metric_Pad1.18x1.45mm_HandSolder
- J2: footprint Connector_Dsub:DSUB-15-HD_Female_Horizontal_P2.29x1.98mm_EdgePinOffset3.03mm_Housed_MountingHolesOffset4.94mm -> Connector_Dsub:DSUB-15_Male_Horizontal_P2.77x2.84mm_EdgePinOffset4.94mm_Housed_MountingHolesOffset7.48mm
- J4, J5: footprint Connector_Wire:SolderWire-0.15sqmm_1x02_P4mm_D0.5mm_OD1.5mm_Relief2x -> Connector_Wire:SolderWire-0.15sqmm_1x02_P4mm_D0.5mm_OD1.5mm
- R1, R2, R3, R4, R5: footprint Resistor_SMD:R_1206_3216Metric_Pad1.42x1.75mm_HandSolder -> Resistor_SMD:R_1206_3216Metric_Pad1.30x1.75mm_HandSolder
- R6, R7: footprint Resistor_SMD:R_0805_2012Metric_Pad1.15x1.40mm_HandSolder -> Resistor_SMD:R_0805_2012Metric_Pad1.20x1.40mm_HandSolder
